Commit message: fix fingers

File: src/lib/assets/G1/G1_hand/urdf/G1_hand.urdf (robot description, URDF)
Before this commit: robot g1_29dof_rev_1_0_with_inspire_hand_DFQ, 63 links, 62 joints
Joints:
- joint L_index_intermediate_joint: type revolute -> fixed
- joint L_index_proximal_joint: type revolute -> fixed
- joint L_middle_intermediate_joint: type revolute -> fixed
- joint L_middle_proximal_joint: type revolute -> fixed
- joint L_pinky_intermediate_joint: type revolute -> fixed
- joint L_pinky_proximal_joint: type revolute -> fixed
- joint L_ring_intermediate_joint: type revolute -> fixed
- joint L_ring_proximal_joint: type revolute -> fixed
- joint L_thumb_distal_joint: type revolute -> fixed
- joint L_thumb_intermediate_joint: type revolute -> fixed
- joint L_thumb_proximal_pitch_joint: type revolute -> fixed
- joint L_thumb_proximal_yaw_joint: type revolute -> fixed
- joint R_index_intermediate_joint: type revolute -> fixed
- joint R_index_proximal_joint: type revolute -> fixed
- joint R_middle_intermediate_joint: type revolute -> fixed
- joint R_middle_proximal_joint: type revolute -> fixed
- joint R_pinky_intermediate_joint: type revolute -> fixed
- joint R_pinky_proximal_joint: type revolute -> fixed
- joint R_ring_intermediate_joint: type revolute -> fixed
- joint R_ring_proximal_joint: type revolute -> fixed
- joint R_thumb_distal_joint: type revolute -> fixed
- joint R_thumb_intermediate_joint: type revolute -> fixed
- joint R_thumb_proximal_pitch_joint: type revolute -> fixed
- joint R_thumb_proximal_yaw_joint: type revolute -> fixed
