Commit message: update joint limit

File: src/lib/assets/GOAT/WF_GOAT/urdf/WF_GOAT.urdf (robot description, URDF)
Before this commit: robot wheel_GOAT, 9 links, 8 joints
Joints:
- joint hip_L_Joint: limit lower=-2.05949 upper=1.09956 effort=4.5 velocity=33.5 -> lower=-1.22173 upper=0.750492 effort=4.5 velocity=15.0
- joint hip_R_Joint: limit lower=-1.09956 upper=2.05949 effort=4.5 velocity=33.5 -> lower=-0.750492 upper=1.22173 effort=4.5 velocity=15.0
- joint knee_L_Joint: limit lower=-0.523599 upper=1.75192 effort=4.5 velocity=33.5 -> lower=0.0 upper=2.30383 effort=4.5 velocity=15
- joint knee_R_Joint: limit lower=-1.75192 upper=0.523599 effort=4.5 velocity=33.5 -> lower=-2.30383 upper=0.0 effort=4.5 velocity=15
- joint thigh_L_Joint: limit lower=-0.593412 upper=1.88496 effort=4.5 velocity=33.5 -> lower=-0.261799 upper=2.05949 effort=4.5 velocity=15.0
- joint thigh_R_Joint: limit lower=-1.88496 upper=0.593412 effort=4.5 velocity=33.5 -> lower=-2.05949 upper=0.261799 effort=4.5 velocity=15.0
- joint wheel_L_Joint: limit lower=-1000000 upper=1000000 effort=2.5 velocity=33.5 -> lower=-1000000 upper=1000000 effort=2.5 velocity=40
- joint wheel_R_Joint: limit lower=-1000000 upper=1000000 effort=2.5 velocity=33.5 -> lower=-1000000 upper=1000000 effort=2.5 velocity=40

Commit message: update mass

File: src/lib/assets/GOAT/WF_GOAT/urdf/WF_GOAT.urdf (robot description, URDF)
Before this commit: robot wheel_GOAT, 9 links, 8 joints
Links:
- link base_Link: mass 2.818 -> 3.075
- link calf_L_Link: mass 0.287 -> 0.321
- link calf_R_Link: mass 0.287 -> 0.321
- link hip_L_Link: mass 0.32 -> 0.316
- link hip_R_Link: mass 0.32 -> 0.316
- link thigh_L_Link: mass 0.429 -> 0.473
- link thigh_R_Link: mass 0.429 -> 0.473
- link wheel_L_Link: mass 0.212 -> 0.238
- link wheel_R_Link: mass 0.212 -> 0.238

Commit message: add imu link

File: src/lib/assets/GOAT/WF_GOAT/urdf/WF_GOAT.urdf (robot description, URDF)
Before this commit: robot wheel_GOAT, 9 links, 8 joints
Links:
- added link imu_link
- link base_Link: mass 3.075 -> 2.818
- link calf_L_Link: mass 0.321 -> 0.287
- link calf_R_Link: mass 0.321 -> 0.287
- link hip_L_Link: mass 0.316 -> 0.32
- link hip_R_Link: mass 0.316 -> 0.32
- link thigh_L_Link: mass 0.473 -> 0.429
- link thigh_R_Link: mass 0.473 -> 0.429
- link wheel_L_Link: mass 0.238 -> 0.212
- link wheel_R_Link: mass 0.238 -> 0.212
Joints:
- added joint imu_joint: type fixed, parent base_Link, child imu_link, origin xyz=0 0 0 rpy=0 0 0
- joint hip_L_Joint: limit lower=-1.22173 upper=0.750492 effort=4.5 velocity=15.0 -> lower=-2.05949 upper=1.09956 effort=4.5 velocity=33.5
- joint hip_R_Joint: limit lower=-0.750492 upper=1.22173 effort=4.5 velocity=15.0 -> lower=-1.09956 upper=2.05949 effort=4.5 velocity=33.5
- joint knee_L_Joint: limit lower=0.0 upper=2.30383 effort=4.5 velocity=15 -> lower=-0.523599 upper=1.75192 effort=4.5 velocity=33.5
- joint knee_R_Joint: limit lower=-2.30383 upper=0.0 effort=4.5 velocity=15 -> lower=-1.75192 upper=0.523599 effort=4.5 velocity=33.5
- joint thigh_L_Joint: limit lower=-0.261799 upper=2.05949 effort=4.5 velocity=15.0 -> lower=-0.593412 upper=1.88496 effort=4.5 velocity=33.5
- joint thigh_R_Joint: limit lower=-2.05949 upper=0.261799 effort=4.5 velocity=15.0 -> lower=-1.88496 upper=0.593412 effort=4.5 velocity=33.5
- joint wheel_L_Joint: limit lower=-1000000 upper=1000000 effort=2.5 velocity=40 -> lower=-1000000 upper=1000000 effort=2.5 velocity=33.5
- joint wheel_R_Joint: limit lower=-1000000 upper=1000000 effort=2.5 velocity=40 -> lower=-1000000 upper=1000000 effort=2.5 velocity=33.5

Commit message: Collision Mesh

File: src/lib/assets/GOAT/WF_GOAT/urdf/WF_GOAT.urdf (robot description, URDF)
Before this commit: robot wheel_GOAT, 10 links, 9 joints
Links:
- link hip_L_Link: geometry collision cylinder length=135E-03 radius=42E-03; visual mesh filename=../meshes/hip_L_Link.stl
- link hip_R_Link: geometry collision cylinder length=135E-03 radius=42E-03; visual mesh filename=../meshes/hip_R_Link.stl
- link thigh_L_Link: geometry collision box size=0.09 0.05 0.145; visual mesh filename=../meshes/thigh_L_Link.stl
- link thigh_R_Link: geometry collision box size=0.09 0.05 0.145; visual mesh filename=../meshes/thigh_R_Link.stl
