Commit message: URDF Mesh-based Collision

File: src/lib/assets/robots/GOAT/WF_GOAT/urdf/WF_GOAT.urdf (robot description, URDF)
Before this commit: robot wheel_GOAT, 10 links, 9 joints
Links:
- link base_Link: geometry collision mesh filename=../meshes/base_Link.stl; visual mesh filename=../meshes/base_Link.stl

Commit message: URDF change

File: src/lib/assets/robots/GOAT/WF_GOAT/urdf/WF_GOAT.urdf (robot description, URDF)
Before this commit: robot wheel_GOAT, 10 links, 9 joints
Links:
- link base_Link: geometry collision box size=0.214 0.200 0.190; visual mesh filename=../meshes/base_Link.stl
Joints:
- joint hip_L_Joint: limit lower=-2.05949 upper=1.09956 effort=4.5 velocity=33.5 -> lower=-1.7453 upper=1.0123 effort=4.5 velocity=33.5
- joint hip_R_Joint: limit lower=-1.09956 upper=2.05949 effort=4.5 velocity=33.5 -> lower=-1.0123 upper=1.7453 effort=4.5 velocity=33.5
- joint knee_L_Joint: limit lower=-0.523599 upper=1.75192 effort=4.5 velocity=33.5 -> lower=-0.523599 upper=2.3387 effort=4.5 velocity=33.5
- joint knee_R_Joint: limit lower=-1.75192 upper=0.523599 effort=4.5 velocity=33.5 -> lower=-2.3387 upper=0.523599 effort=4.5 velocity=33.5
- joint thigh_L_Joint: limit lower=-0.593412 upper=1.88496 effort=4.5 velocity=33.5 -> lower=-0.3840 upper=2.0071 effort=4.5 velocity=33.5
- joint thigh_R_Joint: limit lower=-1.88496 upper=0.593412 effort=4.5 velocity=33.5 -> lower=-2.0071 upper=0.3840 effort=4.5 velocity=33.5
