Commit message: GOAT URDF

File: src/lib/assets/robots/GOAT/WF_GOAT/urdf/WF_GOAT.urdf (robot description, URDF)
Before this commit: robot wheel_GOAT, 10 links, 9 joints
Links:
- link calf_L_Link: mass 0.287 -> 0.299
- link calf_R_Link: mass 0.287 -> 0.299
- link thigh_L_Link: mass 0.429 -> 0.483
- link thigh_R_Link: mass 0.429 -> 0.483

Commit message: URDF update

File: src/lib/assets/robots/GOAT/WF_GOAT/urdf/WF_GOAT.urdf (robot description, URDF)
Before this commit: robot wheel_GOAT, 10 links, 9 joints
Links:
- link base_Link: mass 2.818 -> 3.119
- link calf_L_Link: mass 0.299 -> 0.326
- link calf_R_Link: mass 0.299 -> 0.327
- link hip_L_Link: mass 0.32 -> 0.316; geometry collision cylinder length=48E-03 radius=43.5E-03; visual mesh filename=../meshes/hip_L_Link.stl
- link hip_R_Link: mass 0.32 -> 0.322; geometry collision cylinder length=48E-03 radius=43.5E-03; visual mesh filename=../meshes/hip_R_Link.stl
- link thigh_L_Link: mass 0.483 -> 0.496; geometry collision cylinder length=266E-03 radius=41E-03; visual mesh filename=../meshes/thigh_L_Link.stl
- link thigh_R_Link: mass 0.483 -> 0.495; geometry collision cylinder length=266E-03 radius=41E-03; visual mesh filename=../meshes/thigh_R_Link.stl
- link wheel_L_Link: mass 0.212 -> 0.239
- link wheel_R_Link: mass 0.212 -> 0.217
Joints:
- joint hip_L_Joint: limit lower=-1.7453 upper=1.0123 effort=4.5 velocity=33.5 -> lower=-2.05949 upper=1.09956 effort=4.5 velocity=33.5
- joint hip_R_Joint: limit lower=-1.0123 upper=1.7453 effort=4.5 velocity=33.5 -> lower=-1.09956 upper=2.05949 effort=4.5 velocity=33.5
- joint knee_L_Joint: limit lower=-0.523599 upper=2.3387 effort=4.5 velocity=33.5 -> lower=-0.523599 upper=1.75192 effort=4.5 velocity=33.5
- joint knee_R_Joint: limit lower=-2.3387 upper=0.523599 effort=4.5 velocity=33.5 -> lower=-1.75192 upper=0.523599 effort=4.5 velocity=33.5
- joint thigh_L_Joint: limit lower=-0.3840 upper=2.0071 effort=4.5 velocity=33.5 -> lower=-0.593412 upper=1.88496 effort=4.5 velocity=33.5
- joint thigh_R_Joint: limit lower=-2.0071 upper=0.3840 effort=4.5 velocity=33.5 -> lower=-1.88496 upper=0.593412 effort=4.5 velocity=33.5

Commit message: URDF

File: src/lib/assets/robots/GOAT/WF_GOAT/urdf/WF_GOAT.urdf (robot description, URDF)
Before this commit: robot wheel_GOAT, 10 links, 9 joints
Links:
- link hip_L_Link: geometry collision cylinder length=135E-03 radius=42E-03; visual mesh filename=../meshes/hip_L_Link.stl
- link hip_R_Link: geometry collision cylinder length=135E-03 radius=42E-03; visual mesh filename=../meshes/hip_R_Link.stl
- link thigh_L_Link: geometry collision box size=0.09 0.05 0.145; visual mesh filename=../meshes/thigh_L_Link.stl
- link thigh_R_Link: geometry collision box size=0.09 0.05 0.145; visual mesh filename=../meshes/thigh_R_Link.stl
Joints:
- joint hip_L_Joint: limit lower=-2.05949 upper=1.09956 effort=4.5 velocity=33.5 -> lower=-1.7453 upper=1.0123 effort=4.5 velocity=33.5
- joint hip_R_Joint: limit lower=-1.09956 upper=2.05949 effort=4.5 velocity=33.5 -> lower=-1.0123 upper=1.7453 effort=4.5 velocity=33.5
- joint knee_L_Joint: limit lower=-0.523599 upper=1.75192 effort=4.5 velocity=33.5 -> lower=-0.523599 upper=2.3387 effort=4.5 velocity=33.5
- joint knee_R_Joint: limit lower=-1.75192 upper=0.523599 effort=4.5 velocity=33.5 -> lower=-2.3387 upper=0.523599 effort=4.5 velocity=33.5
- joint thigh_L_Joint: limit lower=-0.593412 upper=1.88496 effort=4.5 velocity=33.5 -> lower=-0.3840 upper=2.0071 effort=4.5 velocity=33.5
- joint thigh_R_Joint: limit lower=-1.88496 upper=0.593412 effort=4.5 velocity=33.5 -> lower=-2.0071 upper=0.3840 effort=4.5 velocity=33.5

Commit message: URDF

File: src/lib/assets/robots/GOAT/WF_GOAT/urdf/WF_GOAT.urdf (robot description, URDF)
Before this commit: robot wheel_GOAT, 10 links, 9 joints
Links:
- link base_Link: geometry collision box size=0.07 0.25 0.08; collision box size=0.214 0.200 0.190

Commit message: Wheel URDF

File: src/lib/assets/robots/GOAT/WF_GOAT/urdf/WF_GOAT.urdf (robot description, URDF)
Before this commit: robot wheel_GOAT, 10 links, 9 joints
Links:
- link wheel_L_Link: geometry collision cylinder length=7E-03 radius=72.75E-03; visual mesh filename=../meshes/wheel_L_Link.stl
- link wheel_R_Link: geometry collision cylinder length=7E-03 radius=72.75E-03; visual mesh filename=../meshes/wheel_R_Link.stl

Commit message: Brand new wheel

File: src/lib/assets/robots/GOAT/WF_GOAT/urdf/WF_GOAT.urdf (robot description, URDF)
Before this commit: robot wheel_GOAT, 10 links, 9 joints
Links:
- link wheel_L_Link: mass 0.239 -> 0.985; geometry collision cylinder length=7E-03 radius=72.75E-03; visual mesh filename=../meshes/New_wheel_L_Link.stl
- link wheel_R_Link: mass 0.217 -> 0.985; geometry collision cylinder length=7E-03 radius=72.75E-03; visual mesh filename=../meshes/New_wheel_R_Link.stl

Commit message: New Wheel URDF

File: src/lib/assets/robots/GOAT/WF_GOAT/urdf/WF_GOAT.urdf (robot description, URDF)
Before this commit: robot wheel_GOAT, 10 links, 9 joints
Links:
- link wheel_L_Link: geometry collision cylinder length=0.05 radius=0.1; visual mesh filename=../meshes/New_wheel_L_Link.stl
- link wheel_R_Link: geometry collision cylinder length=0.05 radius=0.1; visual mesh filename=../meshes/New_wheel_R_Link.stl

Commit message: URDF

File: src/lib/assets/robots/GOAT/WF_GOAT/urdf/WF_GOAT.urdf (robot description, URDF)
Before this commit: robot wheel_GOAT, 10 links, 9 joints
Links:
- link base_Link: mass 3.119 -> 3.153308
- link calf_L_Link: mass 0.326 -> 0.303
- link calf_R_Link: mass 0.327 -> 0.303
- link hip_L_Link: mass 0.316 -> 0.319
- link hip_R_Link: mass 0.322 -> 0.319
- link thigh_L_Link: mass 0.496 -> 0.483216
- link thigh_R_Link: mass 0.495 -> 0.483216
Joints:
- joint hip_L_Joint: origin xyz=38.386E-03 94.233E-03 -152.597E-03 rpy=0 0 0 -> xyz=49.579E-03 96.336E-03 -87.088E-03 rpy=0 0 0
- joint hip_R_Joint: origin xyz=38.386E-03 -94.233E-03 -152.597E-03 rpy=0 0 0 -> xyz=49.579E-03 -96.336E-03 -87.088E-03 rpy=0 0 0

Commit message: .

File: src/lib/assets/robots/GOAT/WF_GOAT/urdf/WF_GOAT.urdf (robot description, URDF)
Before this commit: robot wheel_GOAT, 10 links, 9 joints
Links:
- link wheel_L_Link: mass 0.985 -> 0.220; geometry collision cylinder length=7E-03 radius=72.75E-03; visual mesh filename=../meshes/wheel_L_Link.stl
- link wheel_R_Link: mass 0.985 -> 0.220; geometry collision cylinder length=7E-03 radius=72.75E-03; visual mesh filename=../meshes/wheel_R_Link.stl

Commit message: New wheel URDF

File: src/lib/assets/robots/GOAT/WF_GOAT/urdf/WF_GOAT.urdf (robot description, URDF)
Before this commit: robot wheel_GOAT, 10 links, 9 joints
Links:
- link wheel_L_Link: mass 0.220 -> 0.985; geometry collision cylinder length=0.05 radius=0.1; visual mesh filename=../meshes/New_wheel_L_Link.stl
- link wheel_R_Link: mass 0.220 -> 0.985; geometry collision cylinder length=0.05 radius=0.1; visual mesh filename=../meshes/New_wheel_R_Link.stl

Commit message: URDF

File: src/lib/assets/robots/GOAT/WF_GOAT/urdf/WF_GOAT.urdf (robot description, URDF)
Before this commit: robot wheel_GOAT, 10 links, 9 joints
Links:
- link hip_L_Link: mass 0.319 -> 0.326
- link hip_R_Link: mass 0.319 -> 0.326

Commit message: URDF Viz

File: src/lib/assets/robots/GOAT/WF_GOAT/urdf/WF_GOAT.urdf (robot description, URDF)
Before this commit: robot wheel_GOAT, 10 links, 9 joints
Joints:
- joint hip_L_Joint: origin xyz=49.579E-03 96.336E-03 -87.088E-03 rpy=0 0 0 -> xyz=51.079E-03 96.336E-03 -87.088E-03 rpy=0 0 0
- joint hip_R_Joint: origin xyz=49.579E-03 -96.336E-03 -87.088E-03 rpy=0 0 0 -> xyz=51.079E-03 -96.336E-03 -87.088E-03 rpy=0 0 0

Commit message: No hip

File: src/lib/assets/robots/GOAT/WF_GOAT/urdf/WF_GOAT.urdf (robot description, URDF)
Before this commit: robot wheel_GOAT, 10 links, 9 joints
Links:
- link base_Link: mass 3.153308 -> 2.804789

Commit message: edit joint

File: src/lib/assets/robots/GOAT/WF_GOAT/urdf/WF_GOAT.urdf (robot description, URDF)
Before this commit: robot wheel_GOAT, 10 links, 9 joints
Joints:
- joint hip_L_Joint: axis -1 0 0 -> (none); limit lower=-1.7453 upper=1.0123 effort=4.5 velocity=33.5 -> (none); origin xyz=51.079E-03 96.336E-03 -87.088E-03 rpy=0 0 0 -> xyz=51.079E-03 96.336E-03 -87.088E-03 rpy=0.034906585 0 0
- joint hip_R_Joint: axis -1 0 0 -> (none); limit lower=-1.0123 upper=1.7453 effort=4.5 velocity=33.5 -> (none); origin xyz=51.079E-03 -96.336E-03 -87.088E-03 rpy=0 0 0 -> xyz=51.079E-03 -96.336E-03 -87.088E-03 rpy=-0.034906585 0 0

Commit message: hip update

File: src/lib/assets/robots/GOAT/WF_GOAT/urdf/WF_GOAT.urdf (robot description, URDF)
Before this commit: robot wheel_GOAT, 10 links, 9 joints
Links:
- link hip_L_Link: mass 0.326 -> 0.321
- link hip_R_Link: mass 0.326 -> 0.321

Commit message: .

File: src/lib/assets/robots/GOAT/WF_GOAT/urdf/WF_GOAT.urdf (robot description, URDF)
Before this commit: robot wheel_GOAT, 10 links, 9 joints
Links:
- link base_Link: geometry collision box size=0.214 0.200 0.185; visual mesh filename=../meshes/base_Link.stl

Commit message: URDF Update

File: src/lib/assets/robots/GOAT/WF_GOAT/urdf/WF_GOAT.urdf (robot description, URDF)
Before this commit: robot wheel_GOAT, 10 links, 9 joints
Links:
- link base_Link: geometry collision box size=0.214 0.200 0.182; visual mesh filename=../meshes/base_Link.stl
- link calf_L_Link: mass 0.303 -> 0.320988
- link calf_R_Link: mass 0.303 -> 0.320988
- link hip_L_Link: mass 0.321 -> 0.320539
- link hip_R_Link: mass 0.321 -> 0.320539
- link thigh_L_Link: mass 0.483216 -> 0.520075
- link thigh_R_Link: mass 0.483216 -> 0.520075

Commit message: .

File: src/lib/assets/robots/GOAT/WF_GOAT/urdf/WF_GOAT.urdf (robot description, URDF)
Before this commit: robot wheel_GOAT, 10 links, 9 joints
Links:
- link base_Link: mass 2.804789 -> 2.810462

Commit message: urdf

File: src/lib/assets/robots/GOAT/WF_GOAT/urdf/WF_GOAT.urdf (robot description, URDF)
Before this commit: robot wheel_GOAT, 10 links, 9 joints
Joints:
- joint hip_L_Joint: origin xyz=51.079E-03 96.336E-03 -87.088E-03 rpy=0.034906585 0 0 -> xyz=57.472E-03 95.508E-03 -101.356E-03 rpy=0.034906585 0 0
- joint hip_R_Joint: origin xyz=51.079E-03 -96.336E-03 -87.088E-03 rpy=-0.034906585 0 0 -> xyz=57.472E-03 -95.508E-03 -101.356E-03 rpy=-0.034906585 0 0

Commit message: .

File: src/lib/assets/robots/GOAT/WF_GOAT/urdf/WF_GOAT.urdf (robot description, URDF)
Before this commit: robot wheel_GOAT, 10 links, 9 joints
Links:
- link calf_L_Link: mass 0.320988 -> 0.326882
- link calf_R_Link: mass 0.320988 -> 0.326882
Joints:
- joint knee_L_Joint: origin xyz=0 18E-03 -205E-03 rpy=0 0 0 -> xyz=0 23E-03 -205E-03 rpy=0 0 0
- joint knee_R_Joint: origin xyz=0 -18E-03 -205E-03 rpy=0 0 0 -> xyz=0 -23E-03 -205E-03 rpy=0 0 0
- joint wheel_L_Joint: origin xyz=0 16.555E-03 -200E-03 rpy=0 0 0 -> xyz=0 20.7E-03 -200E-03 rpy=0 0 0
- joint wheel_R_Joint: origin xyz=0 -16.555E-03 -200E-03 rpy=0 0 0 -> xyz=0 -20.7E-03 -200E-03 rpy=0 0 0

Commit message: .

File: src/lib/assets/robots/GOAT/WF_GOAT/urdf/WF_GOAT.urdf (robot description, URDF)
Before this commit: robot wheel_GOAT, 10 links, 9 joints
Links:
- link wheel_L_Link: geometry collision cylinder length=0.05 radius=0.09375; visual mesh filename=../meshes/BF_wheel_L_Link.stl
- link wheel_R_Link: geometry collision cylinder length=0.05 radius=0.09375; visual mesh filename=../meshes/BF_wheel_R_Link.stl

Commit message: .

File: src/lib/assets/robots/GOAT/WF_GOAT/urdf/WF_GOAT.urdf (robot description, URDF)
Before this commit: robot wheel_GOAT, 10 links, 9 joints
Links:
- link wheel_L_Link: geometry collision cylinder length=0.05 radius=0.095; visual mesh filename=../meshes/BF_wheel_L_Link.stl
- link wheel_R_Link: geometry collision cylinder length=0.05 radius=0.095; visual mesh filename=../meshes/BF_wheel_R_Link.stl
