Commit message: Locomotion PF

File: src/lib/assets/robots/GOAT/PF_GOAT/urdf/PF_GOAT.urdf (robot description, URDF)
Before this commit: robot point_GOAT, 8 links, 7 joints
Links:
- link calf_L_Link: geometry collision cylinder length=180E-03 radius=30.0E-03; collision sphere radius=35E-03
- link calf_R_Link: geometry collision cylinder length=180E-03 radius=30.0E-03; collision sphere radius=35E-03

Commit message: new urdf

File: src/lib/assets/robots/GOAT/PF_GOAT/urdf/PF_GOAT.urdf (robot description, URDF)
Before this commit: robot point_GOAT, 8 links, 7 joints
Links:
- link base_Link: mass 3.119 -> 3.153308; geometry collision box size=0.07 0.25 0.08; collision box size=0.214 0.200 0.190
- link hip_L_Link: mass 0.316 -> 0.319
- link hip_R_Link: mass 0.322 -> 0.319
- link thigh_L_Link: mass 0.496 -> 0.483216
- link thigh_R_Link: mass 0.495 -> 0.483216
Joints:
- removed joint thigh_R_Joint
- joint hip_L_Joint: origin xyz=38.386E-03 94.233E-03 -152.597E-03 rpy=0 0 0 -> xyz=49.579E-03 96.336E-03 -87.088E-03 rpy=0 0 0
- joint hip_R_Joint: origin xyz=38.386E-03 -94.233E-03 -152.597E-03 rpy=0 0 0 -> xyz=49.579E-03 -96.336E-03 -87.088E-03 rpy=0 0 0

File: src/lib/assets/robots/GOAT/WF_GOAT/urdf/WF_GOAT.urdf (robot description, URDF)
Before this commit: robot wheel_GOAT, 10 links, 9 joints
Links:
- link wheel_L_Link: geometry collision cylinder length=0.05 radius=0.1; visual mesh filename=../meshes/BF_wheel_L_Link.stl
- link wheel_R_Link: geometry collision cylinder length=0.05 radius=0.1; visual mesh filename=../meshes/BF_wheel_R_Link.stl

Commit message: gear ratio

File: src/lib/assets/robots/GOAT/PF_GOAT/urdf/PF_GOAT.urdf (robot description, URDF)
Before this commit: robot point_GOAT, 8 links, 6 joints
Joints:
- joint knee_L_Joint: limit lower=-0.523599 upper=2.3387 effort=4.5 velocity=33.5 -> lower=-0.523599 upper=2.3387 effort=9.0 velocity=33.5
- joint knee_R_Joint: limit lower=-2.3387 upper=0.523599 effort=4.5 velocity=33.5 -> lower=-2.3387 upper=0.523599 effort=9.0 velocity=33.5

File: src/lib/assets/robots/GOAT/WF_GOAT/urdf/WF_GOAT.urdf (robot description, URDF)
Before this commit: robot wheel_GOAT, 10 links, 9 joints
Joints:
- joint knee_L_Joint: limit lower=-0.523599 upper=2.3387 effort=4.5 velocity=33.5 -> lower=-0.523599 upper=2.3387 effort=9.0 velocity=33.5
- joint knee_R_Joint: limit lower=-2.3387 upper=0.523599 effort=4.5 velocity=33.5 -> lower=-2.3387 upper=0.523599 effort=9.0 velocity=33.5
