Commit message: G1 update

File: src/lib/assets/robots/G1/urdf/G1_standard.urdf (robot description, URDF)
Before this commit: robot g1_standard, 38 links, 37 joints
Links:
- added link pelvis_contour_link, mass 0.001; collision mesh filename=meshes/pelvis_contour_link.STL; visual mesh filename=meshes/pelvis_contour_link.STL
- link pelvis: geometry visual mesh filename=meshes/pelvis_ver0529.STL
Joints:
- added joint pelvis_contour_joint: type fixed, parent pelvis, child pelvis_contour_link
